Commit message: fix some bugs

File: crazydog_ws/src/qlr_control/qlr_control/robot_models/big bipedal robot v1/urdf/big bipedal robot v1.urdf (robot description, URDF)
Before this commit: robot big bipedal robot v1, 10 links, 9 joints
Links:
- link wheelL_link: mass 0.695 -> 0.0
- link wheelR_link: mass 0.695 -> 0.0
